File: MammothMIDI_Circuit/MammothMIDI.sch (KiCad schematic (older format))
At the start: 17 parts, among them SW1 SW_SPST, SW2 SW_SPST, SW3 SW_SPST, SW4 SW_SPST, SW5 SW_SPST, SW6 SW_SPST, U1 TCA9548APWR

Commit message: checkpoint
Parts:
- removed DS? (x2): SSH1106_128X64, symbol MammothMIDI_Library:SSH1106_128X64
- removed SW?: Rotary_Encoder_Switch, symbol Device:Rotary_Encoder_Switch
- added J1: Jack-DC, symbol Connector:Jack-DC
- added J2: DIN-5, symbol Connector:DIN-5_180degree
- added R1, R2: 220Ω, symbol Device:R
Connections:
- net GND: now also DS3.0 (GND), DS4.0 (GND), J1.1, J2.2
- net VCC: now also DS3.1 (VCC), DS4.1 (VCC)
- net at A1.1 (D1/TX): now also R2.1
- net at A1.27 (+5V): now also R1.1
- net at A1.30 (VIN): now also J1.2
- new net: J2.4, R1.2
- new net: J2.5, R2.2
Changed lines of the file:
@@
 $EndDescr
-$Comp
-L MCU_Module:Arduino_Nano_v3.x A1
-U 1 1 5D09ADC7
-P 4800 3750
-F 0 "A1" H 4800 2661 50  0000 C CNN
-F 1 "Arduino_Nano_v3.x" H 4800 2570 50  0000 C CNN
-F 2 "Module:Arduino_Nano" H 4950 2800 50  0001 L CNN
-F 3 "http://www.mouser.com/pdfdocs/Gravitech_Arduino_Nano3_0.pdf" H 4800 2750 50  0001 C CNN
-	1    4800 3750
-	1    0    0    -1
-$EndComp
 $Comp
 L Interface_Expansion:TCA9548APWR U1
@@
 L power:GND #PWR?
 U 1 1 5D0AD602
-P 10500 2750
-F 0 "#PWR?" H 10500 2500 50  0001 C CNN
-F 1 "GND" H 10505 2577 50  0000 C CNN
-F 2 "" H 10500 2750 50  0001 C CNN
-F 3 "" H 10500 2750 50  0001 C CNN
-	1    10500 2750
+P 10500 2700
+F 0 "#PWR?" H 10500 2450 50  0001 C CNN
+F 1 "GND" H 10505 2527 50  0000 C CNN
+F 2 "" H 10500 2700 50  0001 C CNN
+F 3 "" H 10500 2700 50  0001 C CNN
+	1    10500 2700
 	1    0    0    -1
 $EndComp
@@
 L power:GND #PWR?
 U 1 1 5D0ADA34
-P 10500 3450
-F 0 "#PWR?" H 10500 3200 50  0001 C CNN
-F 1 "GND" H 10505 3277 50  0000 C CNN
-F 2 "" H 10500 3450 50  0001 C CNN
-F 3 "" H 10500 3450 50  0001 C CNN
-	1    10500 3450
+P 10500 3400
+F 0 "#PWR?" H 10500 3150 50  0001 C CNN
+F 1 "GND" H 10505 3227 50  0000 C CNN
+F 2 "" H 10500 3400 50  0001 C CNN
+F 3 "" H 10500 3400 50  0001 C CNN
+	1    10500 3400
 	1    0    0    -1
 $EndComp
@@
 L power:VCC #PWR?
 U 1 1 5D0AFFFB
-P 10500 2650
-F 0 "#PWR?" H 10500 2500 50  0001 C CNN
-F 1 "VCC" V 10517 2778 50  0000 L CNN
-F 2 "" H 10500 2650 50  0001 C CNN
-F 3 "" H 10500 2650 50  0001 C CNN
-	1    10500 2650
+P 10500 2600
+F 0 "#PWR?" H 10500 2450 50  0001 C CNN
+F 1 "VCC" V 10517 2728 50  0000 L CNN
+F 2 "" H 10500 2600 50  0001 C CNN
+F 3 "" H 10500 2600 50  0001 C CNN
+	1    10500 2600
 	0    1    1    0
 $EndComp
@@
 L power:VCC #PWR?
 U 1 1 5D0B0D2D
-P 10500 3350
-F 0 "#PWR?" H 10500 3200 50  0001 C CNN
-F 1 "VCC" V 10517 3478 50  0000 L CNN
-F 2 "" H 10500 3350 50  0001 C CNN
-F 3 "" H 10500 3350 50  0001 C CNN
-	1    10500 3350
+P 10500 3300
+F 0 "#PWR?" H 10500 3150 50  0001 C CNN
+F 1 "VCC" V 10517 3428 50  0000 L CNN
+F 2 "" H 10500 3300 50  0001 C CNN
+F 3 "" H 10500 3300 50  0001 C CNN
+	1    10500 3300
 	0    1    1    0
 $EndComp
@@
 	1    0    0    -1
 $EndComp
-$Comp
-L MammothMIDI_Library:SSH1106_128X64 DS?
-U 1 1 5D0BAD80
-P 10150 5450
-F 0 "DS?" H 10150 5765 50  0000 C CNN
-F 1 "SSH1106_128X64" H 10150 5674 50  0000 C CNN
-F 2 "" H 10200 5500 50  0001 C CNN
-F 3 "" H 10200 5500 50  0001 C CNN
-	1    10150 5450
-	1    0    0    -1
-$EndComp
-$Comp
-L MammothMIDI_Library:SSH1106_128X64 DS?
-U 1 1 5D0BB1AA
-P 10150 6150
-F 0 "DS?" H 10150 6465 50  0000 C CNN
-F 1 "SSH1106_128X64" H 10150 6374 50  0000 C CNN
-F 2 "" H 10200 6200 50  0001 C CNN
-F 3 "" H 10200 6200 50  0001 C CNN
-	1    10150 6150
-	1    0    0    -1
-$EndComp
 Wire Wire Line
 	9800 3400 9700 3400
@@
 Wire Wire Line
 	9400 4050 8550 4050
-Wire Wire Line
-	9800 5400 9300 5400
-Wire Wire Line
-	9300 5400 9300 4150
-Wire Wire Line
-	9300 4150 8550 4150
-Wire Wire Line
-	9800 5500 9200 5500
-Wire Wire Line
-	9200 5500 9200 4250
-Wire Wire Line
-	9200 4250 8550 4250
-Wire Wire Line
-	9800 6100 9100 6100
-Wire Wire Line
-	9100 6100 9100 4350
-Wire Wire Line
-	9100 4350 8550 4350
-Wire Wire Line
-	9800 6200 9000 6200
-Wire Wire Line
-	9000 6200 9000 4450
-Wire Wire Line
-	9000 4450 8550 4450
 Wire Wire Line
 	5300 4150 6600 4150
@@
 	3150 5200 3150 5350
 $Comp
-L Device:Rotary_Encoder_Switch SW?
-U 1 1 5D14507E
-P 2550 2850
-F 0 "SW?" H 2550 3217 50  0000 C CNN
-F 1 "Rotary_Encoder_Switch" H 2550 3126 50  0000 C CNN
-F 2 "" H 2400 3010 50  0001 C CNN
-F 3 "~" H 2550 3110 50  0001 C CNN
-	1    2550 2850
-	1    0    0    -1
+L Connector:Jack-DC J1
+U 1 1 5D2757EC
+P 4000 1400
+F 0 "J1" H 3771 1358 50  0000 R CNN
+F 1 "Jack-DC" H 3771 1449 50  0000 R CNN
+F 2 "" H 4050 1360 50  0001 C CNN
+F 3 "~" H 4050 1360 50  0001 C CNN
+	1    4000 1400
+	1    0    0    1
+$EndComp
+$Comp
+L power:GND #PWR?
+U 1 1 5D27C7E4
+P 4450 1600
+F 0 "#PWR?" H 4450 1350 50  0001 C CNN
+F 1 "GND" H 4455 1427 50  0000 C CNN
+F 2 "" H 4450 1600 50  0001 C CNN
+F 3 "" H 4450 1600 50  0001 C CNN
+	1    4450 1600
+	1    0    0    -1
+$EndComp
+Wire Wire Line
+	4300 1300 4700 1300
+Wire Wire Line
+	4300 1500 4450 1500
+Wire Wire Line
+	4450 1500 4450 1600
+$Comp
+L Device:R R1
+U 1 1 5D29F209
+P 3600 2450
+F 0 "R1" V 3393 2450 50  0000 C CNN
+F 1 "220Ω" V 3484 2450 50  0000 C CNN
+F 2 "" V 3530 2450 50  0001 C CNN
+F 3 "~" H 3600 2450 50  0001 C CNN
+	1    3600 2450
+	0    1    1    0
+$EndComp
+$Comp
+L MCU_Module:Arduino_Nano_v3.x A1
+U 1 1 5D09ADC7
+P 4800 3750
+F 0 "A1" H 4800 2661 50  0000 C CNN
+F 1 "Arduino_Nano_v3.x" H 4800 2570 50  0000 C CNN
+F 2 "Module:Arduino_Nano" H 4950 2800 50  0001 L CNN
+F 3 "http://www.mouser.com/pdfdocs/Gravitech_Arduino_Nano3_0.pdf" H 4800 2750 50  0001 C CNN
+	1    4800 3750
+	1    0    0    -1
+$EndComp
+Wire Wire Line
+	4700 1300 4700 2750
+Wire Wire Line
+	3050 2450 3450 2450
+Wire Wire Line
+	3750 2450 5000 2450
+Wire Wire Line
+	5000 2450 5000 2750
+$Comp
+L Device:R R2
+U 1 1 5D2B8A23
+P 3600 3250
+F 0 "R2" V 3393 3250 50  0000 C CNN
+F 1 "220Ω" V 3484 3250 50  0000 C CNN
+F 2 "" V 3530 3250 50  0001 C CNN
+F 3 "~" H 3600 3250 50  0001 C CNN
+	1    3600 3250
+	0    1    1    0
+$EndComp
+Wire Wire Line
+	3750 3250 4300 3250
+Wire Wire Line
+	2450 2450 2200 2450
+Wire Wire Line
+	2200 2450 2200 3250
+Wire Wire Line
+	2200 3250 3450 3250
+$Comp
+L power:GND #PWR?
+U 1 1 5D2BE580
+P 2450 2000
+F 0 "#PWR?" H 2450 1750 50  0001 C CNN
+F 1 "GND" H 2455 1827 50  0000 C CNN
+F 2 "" H 2450 2000 50  0001 C CNN
+F 3 "" H 2450 2000 50  0001 C CNN
+	1    2450 2000
+	1    0    0    -1
+$EndComp
+Wire Wire Line
+	2450 2000 2450 1900
+Wire Wire Line
+	2450 1900 2750 1900
+Wire Wire Line
+	2750 1900 2750 2250
+$Comp
+L Connector:DIN-5_180degree J2
+U 1 1 5D27EBAE
+P 2750 2550
+F 0 "J2" H 2750 2275 50  0000 C CNN
+F 1 "DIN-5" H 2750 2184 50  0000 C CNN
+F 2 "" H 2750 2550 50  0001 C CNN
+F 3 "http://www.mouser.com/ds/2/18/40_c091_abd_e-75918.pdf" H 2750 2550 50  0001 C CNN
+	1    2750 2550
+	-1   0    0    -1
 $EndComp
 $EndSCHEMATC
